File: PSU.kicad_sch (KiCad schematic)
At the start: 104 parts, among them J18 USB_C_Receptacle_USB2.0, J78 Screw_Terminal_01x02, Q5 2N7002, Q6 2N7002, Q7 NCE30P28Q, Q8 2N7002, SW1 SW_Push, SW2 SW_Push, U13 TL431DBZ, U14 CH224K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

Commit message: Initial commit
Parts:
- added C110: 4.7uF, Capacitor_SMD:C_1206_3216Metric, symbol Device:C
- added C111, C112, C113: 22uF, Capacitor_SMD:C_1210_3225Metric, symbol Device:C
- added C99: 22uF, Capacitor_SMD:C_1210_3225Metric_Pad1.33x2.70mm_HandSolder, symbol Device:C
- added F81: 32V/6A, Fuse:Fuse_1206_3216Metric, symbol Device:Fuse
- added F82: Fuse, Fuse:Fuse_1206_3216Metric, symbol Device:Fuse
- added TP16: TestPoint, A_HDJ_Library:TestPoint_Pad_D1.5mm, symbol Connector:TestPoint
- C102: renamed from C?; value C -> 22uF; footprint (none) -> Capacitor_SMD:C_1210_3225Metric_Pad1.33x2.70mm_HandSolder
- C103: renamed from C?; value C -> 4.7uF; footprint (none) -> Capacitor_SMD:C_0805_2012Metric
- C104: renamed from C?; value C -> 1nF; footprint (none) -> Capacitor_SMD:C_0805_2012Metric
- C105: renamed from C?; value C -> 150nF; footprint (none) -> A_HDJ_Library:C_0603_1608Metric
- C106: renamed from C?; value C -> 10uF; footprint (none) -> Capacitor_SMD:C_1210_3225Metric_Pad1.33x2.70mm_HandSolder
- C107: renamed from C?; value C -> 22nF; footprint (none) -> Capacitor_SMD:C_0402_1005Metric
- C108, C109: renamed from C?; value C -> 4.7uF; footprint (none) -> Capacitor_SMD:C_1206_3216Metric
- C72, C73, R50, R56: now fitted; now in the parts list
- L78: renamed from L?; value L -> 560nF; footprint (none) -> XAL6030561MEB:XAL6030561MEB
- Q78: renamed from Q?; footprint SI4427BDY-T1-E3:SOIC127P600X175-8N -> SI4427BDY:SOIC127P600X175-8N
- R81: renamed from R?; value R -> 140k; footprint (none) -> A_HDJ_Library:R_0402_1005Metric
- R84: renamed from R?; value R -> 56.2k; footprint (none) -> A_HDJ_Library:R_0603_1608Metric
- R85: renamed from R?; value R -> 28.7k; footprint (none) -> A_HDJ_Library:R_0603_1608Metric
- R86: renamed from R?; value R -> 178k; footprint (none) -> A_HDJ_Library:R_0402_1005Metric
- R87: renamed from R?; value R -> 732k; footprint (none) -> A_HDJ_Library:R_0402_1005Metric
- R88: renamed from R?; value R -> 80.6k; footprint (none) -> Resistor_SMD:R_0402_1005Metric
- U79: renamed from U?; footprint RNW0013A -> boostTPS:RNW0013A
Connections:
- net +12V: now also C110.2, C111.2, C112.2, C113.2, F82.1, F82.2, TP16.1
- net GND: now also C110.1, C111.1, C112.1, C113.1, C99.1
- net at C107.2, Q78.4, R86.2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: no longer R87.2, R88.1
- net at C102.2, L78.1, U79.11 (EN)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: now also C99.2, F81.2; no longer J78.1 (Pin_1)
- net at U79.5 (FB): now also R87.2, R88.1
- new net: F81.1, J78.1 (Pin_1)
Other:
- moved on the sheet: C102, C103, C104, C105, C106, C107, C108, C109, C61, C62, C63, C64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
