File: PSU.kicad_sch (KiCad schematic)
At the start: 112 parts, among them J18 USB_C_Receptacle_USB2.0, J78 Screw_Terminal_01x02, Q5 2N7002, Q6 2N7002, Q7 NCE30P28Q, Q78 SI4427BDY-T1-E3, Q8 2N7002, SW1 SW_Push, SW2 SW_Push, U13 TL431DBZ, U14 CH224K, U15 SY8253ADC, U16 SY8253ADC, U79 TPS61178RNWR

Commit message: Update KiCad carrier board project
Parts:
- removed C61, C62, C63: 1uF/16V, A_HDJ_Library:C_0402_1005Metric, symbol Device:C
- removed D10, D11: ESD5V0B03, A_HDJ_Library:D_0402_1005Metric, symbol Diode:ESD9B5.0ST5G
- removed D12, D13, D14: PESD24VS1UL-N, A_HDJ_Library:D_0402_1005Metric, symbol Device:D_Zener
- removed D18, D19, D20: SS54, A_HDJ_Library:D_SMA, symbol Device:D_Schottky
- removed D23: LED_G, A_HDJ_Library:LED_0603_1608Metric, symbol Device:LED
- removed J18: USB_C_Receptacle_USB2.0, A_HDJ_Library:USB_C_Receptacle_G-Switch_GT-USB-7010ASV, symbol Connector:USB_C_Receptacle_USB2.0_16P
- removed Q5, Q6: 2N7002, A_HDJ_Library:SOT-23, symbol Transistor_FET:2N7002
- removed Q7: NCE30P28Q, A_HDJ_Library:MOSFET_PDFN8_3.3x3.3, symbol A_HDJ_Library:AON7262E
- removed R36, R38, R40: 10K/1%, A_HDJ_Library:R_0402_1005Metric, symbol Device:R
- removed R37: 1K/1%, A_HDJ_Library:R_0402_1005Metric, symbol Device:R
- removed R39: 2.2K/1%, A_HDJ_Library:R_0402_1005Metric, symbol Device:R
- removed R41, R42, R54: 21.5K/1%, A_HDJ_Library:R_0402_1005Metric, symbol Device:R
- removed R43: 56K/1%, A_HDJ_Library:R_0402_1005Metric, symbol Device:R
- removed R44, R45: 100K/1%, A_HDJ_Library:R_0402_1005Metric, symbol Device:R
- removed TP10, TP3, TP4, TP8, TP9: TestPoint, A_HDJ_Library:TestPoint_Pad_D1.5mm, symbol Connector:TestPoint
- removed U13: TL431DBZ, A_HDJ_Library:SOT-23, symbol Reference_Voltage:TL431DBZ
- removed U14: CH224K, A_HDJ_Library:ESSOP-10-1EP_3.9x5mm_P1.0mm_EP3.2x2.3, symbol A_HDJ_Library:CH224K
Connections:
- no-connect marks 5 -> 0
Other:
- note removed: "15V PD Input"
- note removed: "CH224K get DC 15V power from USB-PD adapter"
- note removed: "PCIe Power Enable LED"
- note removed: "PWR_C_D+"
- note removed: "PWR_C_D-"
- note removed: "Power for PCIe x4 OVP@13.86V"
- note removed: "soft start"
- company: DFRobot -> (none)
- title: Primer Carrier for LattePanda Mu -> Carrier for LattePanda Mu
