File: USB2.0&USB3.0.kicad_sch (KiCad schematic)
At the start: 53 parts, among them J4 USB3_A_Stacked, J5 USB_A_Stacked, J79 SS-52000-004, J80 0483930003, J81 DX07S024JJ3R1300, J82 USB-A1HSW6, J83 DX07S024JJ4R1300, U4 ULC0524P, U5 ULC0524P, U78 ULC0524P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

Commit message: Initial commit
Parts:
- J80: footprint usba_molex:MOLEX_0483930003 -> revised_usba3:484050003_MOL
Changed lines of the file:
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@@
 			)
 		)
-		(property "Footprint" "usba_molex:MOLEX_0483930003"
+		(property "Footprint" "revised_usba3:484050003_MOL"
 			(at 133.35 180.34 0)
 			(effects
