File: USB2.0&USB3.0.kicad_sch (KiCad schematic)
At the start: 53 parts, among them J4 USB3_A_Stacked, J5 USB_A_Stacked, J79 SS-52000-004, J80 0483930003, J81 DX07S024JJ3R1300, J82 USB-A1HSW6, J83 DX07S024JJ4R1300, U4 ULC0524P, U5 ULC0524P, U78 ULC0524P, U80 ULC0524P, U86 HD3SS3220IRNHT, U90 ULC0524P

Commit message: Update KiCad carrier board project
Parts:
- removed C26, C27, C28, C29, C90, C91, C97, C98: 100nF/50V, A_HDJ_Library:C_0402_1005Metric, symbol Device:C
- removed C32, C87, C95: 22uF/10V, A_HDJ_Library:C_0603_1608Metric, symbol Device:C
- removed D5, D6, D7, D8: ESD5V0B03, A_HDJ_Library:D_0402_1005Metric, symbol Diode:ESD9B5.0ST5G
- removed F5, F80: 6V/2A, A_HDJ_Library:Fuse_0805_2012Metric, symbol Device:Fuse
- removed F78: 6V/2A, A_HDJ_Library:R_0805_2012Metric, symbol Device:Fuse
- removed J4: USB3_A_Stacked, A_HDJ_Library:USB3_A_Molex_48406-0001_Horizontal_Stacked, symbol Connector:USB3_A_Stacked
- removed J5: USB_A_Stacked, A_HDJ_Library:USB_A_CUI_UJ2-ADH-TH_Horizontal_Stacked, symbol Connector:USB_A_Stacked
- removed J79: SS-52000-004, SS-52000-004:BEL_SS-52000-004, symbol SS-52000-004:SS-52000-004
- removed J83: DX07S024JJ4R1300, USBC3.0_good:JAE_DX07S024JJ3R1300, symbol DX07S024JJ4R1300:DX07S024JJ4R1300
- removed R80, R82, R83: 5.1k, A_HDJ_Library:R_0402_1005Metric, symbol Device:R
- removed U4, U5: ULC0524P, A_HDJ_Library:Diodes_UDFN-10_1.0x2.5mm_P0.5mm, symbol Power_Protection:D3V3XA4B10LP
Connections:
- no-connect marks 5 -> 3
Other:
- note removed: "SSRXx_N"
- note removed: "SSRXx_P"
- note removed: "SSTXx_N"
- note removed: "SSTXx_P"
- note removed: "USB_2_P+"
- note removed: "USB_2_P-"
- company: DFRobot -> (none)
- title: Primer Carrier for LattePanda Mu -> Carrier for LattePanda Mu
- moved on the sheet: C100, C101, C86, C88, C89, C92, C93, C94, C96, D78, D79, D80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
