File: fan_temp.kicad_sch (KiCad schematic)
At the start: 23 parts, among them M1 Fan_4pin, M2 Fan_4pin

Commit message: Initial commit
Parts:
- R64, R66: now fitted; now in the parts list
Changed lines of the file:
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@@
 		(unit 1)
 		(exclude_from_sim no)
-		(in_bom no)
+		(in_bom yes)
 		(on_board yes)
-		(dnp yes)
+		(dnp no)
 		(property "Reference" "R66"
 			(at 306.07 175.26 0)
@@
 		(unit 1)
 		(exclude_from_sim no)
-		(in_bom no)
+		(in_bom yes)
 		(on_board yes)
-		(dnp yes)
+		(dnp no)
 		(property "Reference" "R64"
 			(at 303.53 153.67 0)
