File: fan_temp.kicad_sch (KiCad schematic)
At the start: 23 parts, among them M1 Fan_4pin, M2 Fan_4pin

Commit message: Update KiCad carrier board project
Parts:
- removed C85: 100nF/50V, Capacitor_SMD:C_0402_1005Metric, symbol Device:C
- removed D27: 1N5819WS, Diode_SMD:D_SOD-323, symbol Diode:1N5819WS
- removed JP2: NTC_Test, Jumper:SolderJumper-2_P1.3mm_Open_RoundedPad1.0x1.5mm, symbol Jumper:SolderJumper_2_Open
- removed M2: Fan_4pin, Connector_JST:JST_PH_B4B-PH-K_1x04_P2.00mm_Vertical, symbol Motor:Fan_4pin
- removed R63: 10K/1%, Resistor_SMD:R_0402_1005Metric, symbol Device:R
- removed R65, R74: 4.7K/1%, Resistor_SMD:R_0402_1005Metric, symbol Device:R
- removed R67, R70: 21.5K/1%, Resistor_SMD:R_0402_1005Metric, symbol Device:R
- removed R71: 100R/1%, Resistor_SMD:R_0402_1005Metric, symbol Device:R
- removed R73, R75: 0R/1%, RES0603, symbol Device:R
- removed TH1: NTC-10K, Resistor_SMD:R_0603_1608Metric, symbol Device:Thermistor_NTC
Other:
- note removed: "SYS FAN"
- company: DFRobot -> (none)
- title: Primer Carrier for LattePanda Mu -> Carrier for LattePanda Mu
