File: HDMI.kicad_sch (KiCad schematic)
At the start: 37 parts, among them J3 HDMI_A, Q1 2N7002, Q2 2SK3018, Q3 2SK3018, Q4 2SK3018, U1 TPAZ1023-04F, U2 TPAZ1023-04F

Commit message: Update KiCad carrier board project
Other:
- company: DFRobot -> (none)
- title: Primer Carrier for LattePanda Mu -> Carrier for LattePanda Mu
- moved on the sheet: U1, U2
Changed lines of the file:
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@@
 	(paper "A2")
 	(title_block
-		(title "Primer Carrier for LattePanda Mu")
-		(date "2024-03-13")
-		(rev "V1.0.0")
-		(company "DFRobot")
+		(title "Carrier for LattePanda Mu")
 	)
 	(junction
@@
 	)
 	(junction
-		(at 336.55 190.5)
+		(at 269.24 81.28)
 		(diameter 0)
 		(color 0 0 0 0)
@@
 	)
 	(junction
-		(at 285.75 185.42)
+		(at 218.44 76.2)
 		(diameter 0)
 		(color 0 0 0 0)
@@
 	)
 	(junction
-		(at 361.95 190.5)
+		(at 294.64 81.28)
 		(diameter 0)
 		(color 0 0 0 0)
 	)
 	(junction
-		(at 311.15 190.5)
+		(at 243.84 81.28)
 		(diameter 0)
 		(color 0 0 0 0)
@@
 	)
 	(junction
-		(at 336.55 185.42)
+		(at 269.24 76.2)
 		(diameter 0)
 		(color 0 0 0 0)
@@
 	)
 	(junction
-		(at 311.15 185.42)
+		(at 243.84 76.2)
 		(diameter 0)
 		(color 0 0 0 0)
@@
 	)
 	(junction
-		(at 285.75 190.5)
+		(at 218.44 81.28)
 		(diameter 0)
 		(color 0 0 0 0)
@@
 	)
 	(junction
-		(at 361.95 185.42)
+		(at 294.64 76.2)
 		(diameter 0)
 		(color 0 0 0 0)
@@
 	(wire
 		(pts
-			(xy 361.95 190.5) (xy 361.95 195.58)
+			(xy 294.64 81.28) (xy 294.64 86.36)
 		)
 		(stroke
@@
 	(wire
 		(pts
-			(xy 285.75 185.42) (xy 285.75 180.34)
+			(xy 218.44 76.2) (xy 218.44 71.12)
 		)
 		(stroke
@@
 	(wire
 		(pts
-			(xy 311.15 185.42) (xy 311.15 180.34)
+			(xy 243.84 76.2) (xy 243.84 71.12)
 		)
 		(stroke
@@
 	(wire
 		(pts
-			(xy 361.95 180.34) (xy 361.95 185.42)
+			(xy 294.64 71.12) (xy 294.64 76.2)
 		)
 		(stroke
@@
 	(wire
 		(pts
-			(xy 311.15 185.42) (xy 322.58 185.42)
+			(xy 243.84 76.2) (xy 255.27 76.2)
 		)
 		(stroke
@@
 	(wire
 		(pts
-			(xy 336.55 190.5) (xy 336.55 195.58)
+			(xy 269.24 81.28) (xy 269.24 86.36)
 		)
 		(stroke
@@
 	(wire
 		(pts
-			(xy 311.15 190.5) (xy 322.58 190.5)
+			(xy 243.84 81.28) (xy 255.27 81.28)
 		)
 		(stroke
@@
 	(wire
 		(pts
-			(xy 361.95 190.5) (xy 373.38 190.5)
+			(xy 294.64 81.28) (xy 306.07 81.28)
 		)
 		(stroke
@@
 	(wire
 		(pts
-			(xy 336.55 180.34) (xy 336.55 185.42)
+			(xy 269.24 71.12) (xy 269.24 76.2)
 		)
 		(stroke
@@
 	(wire
 		(pts
-			(xy 275.59 185.42) (xy 285.75 185.42)
+			(xy 208.28 76.2) (xy 218.44 76.2)
 		)
 		(stroke
@@
 	(wire
 		(pts
-			(xy 311.15 195.58) (xy 311.15 190.5)
+			(xy 243.84 86.36) (xy 243.84 81.28)
 		)
 		(stroke
@@
 	(wire
 		(pts
-			(xy 326.39 190.5) (xy 336.55 190.5)
+			(xy 259.08 81.28) (xy 269.24 81.28)
 		)
 		(stroke
@@
 	(wire
 		(pts
-			(xy 326.39 185.42) (xy 336.55 185.42)
+			(xy 259.08 76.2) (xy 269.24 76.2)
 		)
 		(stroke
@@
 	(wire
 		(pts
-			(xy 275.59 190.5) (xy 285.75 190.5)
+			(xy 208.28 81.28) (xy 218.44 81.28)
 		)
 		(stroke
@@
 	(wire
 		(pts
-			(xy 285.75 195.58) (xy 285.75 190.5)
+			(xy 218.44 86.36) (xy 218.44 81.28)
 		)
 		(stroke
@@
 	(wire
 		(pts
-			(xy 373.38 185.42) (xy 361.95 185.42)
+			(xy 306.07 76.2) (xy 294.64 76.2)
 		)
 		(stroke
@@
 	)
 	(label "TMDS_D2-"
-		(at 275.59 190.5 0)
+		(at 208.28 81.28 0)
 		(effects
 			(font
@@
 	)
 	(label "TMDS_D0-"
-		(at 326.39 190.5 0)
+		(at 259.08 81.28 0)
 		(effects
 			(font
@@
 	)
 	(label "TMDS_D0+"
-		(at 326.39 185.42 0)
+		(at 259.08 76.2 0)
 		(effects
 			(font
@@
 	)
 	(label "TMDS_D2+"
-		(at 275.59 185.42 0)
+		(at 208.28 76.2 0)
 		(effects
 			(font
@@
 	)
 	(label "TMDS_CK+"
-		(at 373.38 185.42 180)
+		(at 306.07 76.2 180)
 		(effects
 			(font
@@
 	)
 	(label "TMDS_CK-"
-		(at 373.38 190.5 180)
+		(at 306.07 81.28 180)
 		(effects
 			(font
@@
 	)
 	(label "TMDS_D1+"
-		(at 322.58 185.42 180)
+		(at 255.27 76.2 180)
 		(effects
 			(font
@@
 	)
 	(label "TMDS_D1-"
-		(at 322.58 190.5 180)
+		(at 255.27 81.28 180)
 		(effects
 			(font
@@
 	(symbol
 		(lib_id "power:GND")
-		(at 349.25 200.66 0)
+		(at 281.94 91.44 0)
 		(unit 1)
 		(exclude_from_sim no)
@@
 		(fields_autoplaced yes)
 		(property "Reference" "#PWR028"
-			(at 349.25 207.01 0)
+			(at 281.94 97.79 0)
 			(effects
 				(font
@@
 		)
 		(property "Value" "GND"
-			(at 349.25 205.74 0)
+			(at 281.94 96.52 0)
 			(effects
 				(font
@@
 		)
 		(property "Footprint" ""
-			(at 349.25 200.66 0)
+			(at 281.94 91.44 0)
 			(effects
 				(font
@@
 		)
 		(property "Datasheet" ""
-			(at 349.25 200.66 0)
+			(at 281.94 91.44 0)
 			(effects
 				(font
@@
 		)
 		(property "Description" ""
-			(at 349.25 200.66 0)
+			(at 281.94 91.44 0)
 			(effects
 				(font
@@
 	(symbol
 		(lib_id "Power_Protection:D3V3XA4B10LP")
-		(at 349.25 187.96 0)
+		(at 281.94 78.74 0)
 		(unit 1)
 		(exclude_from_sim no)
@@
 		(dnp no)
 		(property "Reference" "U2"
-			(at 354.33 203.2 0)
+			(at 287.02 93.98 0)
 			(effects
 				(font
@@
 		)
 		(property "Value" "TPAZ1023-04F"
-			(at 360.68 200.66 0)
+			(at 293.37 91.44 0)
 			(effects
 				(font
@@
 		)
 		(property "Footprint" "A_HDJ_Library:Diodes_UDFN-10_1.0x2.5mm_P0.5mm"
-			(at 325.12 198.12 0)
+			(at 257.81 88.9 0)
 			(effects
 				(font
@@
 		)
 		(property "Datasheet" "https://www.diodes.com/assets/Datasheets/D3V3XA4B10LP.pdf"
-			(at 349.25 187.96 0)
+			(at 281.94 78.74 0)
 			(effects
 				(font
@@
 		)
 		(property "Description" ""
-			(at 349.25 187.96 0)
+			(at 281.94 78.74 0)
 			(effects
 				(font
@@
 		)
 		(property "SCH_Show_Footprint" ""
-			(at 349.25 187.96 0)
+			(at 281.94 78.74 0)
 			(effects
 				(font
@@
 		)
 		(property "Sim.Device" ""
-			(at 349.25 187.96 0)
+			(at 281.94 78.74 0)
 			(effects
 				(font
@@
 		)
 		(property "Sim.Pins" ""
-			(at 349.25 187.96 0)
+			(at 281.94 78.74 0)
 			(effects
 				(font
@@
 		)
 		(property "Sim.Type" ""
-			(at 349.25 187.96 0)
+			(at 281.94 78.74 0)
 			(effects
 				(font
@@
 	(symbol
 		(lib_id "Power_Protection:D3V3XA4B10LP")
-		(at 298.45 187.96 0)
+		(at 231.14 78.74 0)
 		(unit 1)
 		(exclude_from_sim no)
@@
 		(dnp no)
 		(property "Reference" "U1"
-			(at 303.53 204.47 0)
+			(at 236.22 95.25 0)
 			(effects
 				(font
@@
 		)
 		(property "Value" "TPAZ1023-04F"
-			(at 308.61 201.93 0)
+			(at 241.3 92.71 0)
 			(effects
 				(font
@@
 		)
 		(property "Footprint" "A_HDJ_Library:Diodes_UDFN-10_1.0x2.5mm_P0.5mm"
-			(at 274.32 198.12 0)
+			(at 207.01 88.9 0)
 			(effects
 				(font
@@
 		)
 		(property "Datasheet" "https://www.diodes.com/assets/Datasheets/D3V3XA4B10LP.pdf"
-			(at 298.45 187.96 0)
+			(at 231.14 78.74 0)
 			(effects
 				(font
@@
 		)
 		(property "Description" ""
-			(at 298.45 187.96 0)
+			(at 231.14 78.74 0)
 			(effects
 				(font
@@
 		)
 		(property "SCH_Show_Footprint" ""
-			(at 298.45 187.96 0)
+			(at 231.14 78.74 0)
 			(effects
 				(font
@@
 		)
 		(property "Sim.Device" ""
-			(at 298.45 187.96 0)
+			(at 231.14 78.74 0)
 			(effects
 				(font
@@
 		)
 		(property "Sim.Pins" ""
-			(at 298.45 187.96 0)
+			(at 231.14 78.74 0)
 			(effects
 				(font
@@
 		)
 		(property "Sim.Type" ""
-			(at 298.45 187.96 0)
+			(at 231.14 78.74 0)
 			(effects
 				(font
@@
 	(symbol
 		(lib_id "power:GND")
-		(at 298.45 200.66 0)
+		(at 231.14 91.44 0)
 		(mirror y)
 		(unit 1)
@@
 		(fields_autoplaced yes)
 		(property "Reference" "#PWR027"
-			(at 298.45 207.01 0)
+			(at 231.14 97.79 0)
 			(effects
 				(font
@@
 		)
 		(property "Value" "GND"
-			(at 298.45 205.74 0)
+			(at 231.14 96.52 0)
 			(effects
 				(font
@@
 		)
 		(property "Footprint" ""
-			(at 298.45 200.66 0)
+			(at 231.14 91.44 0)
 			(effects
 				(font
@@
 		)
 		(property "Datasheet" ""
-			(at 298.45 200.66 0)
+			(at 231.14 91.44 0)
 			(effects
 				(font
@@
 		)
 		(property "Description" ""
-			(at 298.45 200.66 0)
+			(at 231.14 91.44 0)
 			(effects
 				(font
