File: LattePanda Module.kicad_sch (KiCad schematic)
At the start: 12 parts, among them J1 Conn_01x03_Pin

Commit message: Update KiCad carrier board project
Other:
- company: DFRobot -> (none)
- title: Primer Carrier for LattePanda Mu -> Carrier for LattePanda Mu
Changed lines of the file:
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@@
 	(paper "A2")
 	(title_block
-		(title "Primer Carrier for LattePanda Mu")
-		(date "2024-04-06")
-		(rev "V1.0.0")
-		(company "DFRobot")
-		(comment 1 "20240406")
+		(title "Carrier for LattePanda Mu")
 	)
 	(text "HSIO functions are defined by the BIOS source code, \nCannot be changed in BIOS settings.\n\nBefore starting design, you should choose one of\nthe available BIOS configurations on:\nhttps://github.com/LattePandaTeam/LattePanda-Mu\nOr contact techsupport for custom your BIOS\n\nThe default functions are defined as follows:\n\n- HSIO0: USB3.2 10Gbps\n- HSIO1: USB3.2 10Gbps\n- HSIO2: PCIe 3.0 x1\n- HSIO3: PCIe 3.0 x1\n\n- HSIO8: PCIe 3.0 x4 (Lane 0)\n- HSIO9: PCIe 3.0 x4 (Lane 1)\n- HSIO10: PCIe 3.0 x4 (Lane 2)\n- HSIO11: PCIe 3.0 x4 (Lane 3)\n\n- HSIO6: PCIe 3.0 x1"
