File: M.2 E&M Key.kicad_sch (KiCad schematic)
At the start: 26 parts, among them J15 Bus_M.2_Socket_M, J16 Bus_M.2_Socket_E

Commit message: Update KiCad carrier board project
Parts:
- removed C49, C50: 220nF/50V, A_HDJ_Library:C_0402_1005Metric, symbol Device:C_Small
- removed C51, C53: 10uF/10V, A_HDJ_Library:C_0402_1005Metric, symbol Device:C
- removed C52, C54: 100nF/50V, A_HDJ_Library:C_0402_1005Metric, symbol Device:C
- removed D9: LED_G, A_HDJ_Library:LED_0603_1608Metric, symbol Device:LED
- removed H8: MountingHole_M2.0, A_HDJ_Library:MountingHole_2.75mm_M2_4.4mm_Pad_TopOnly, symbol Mechanical:MountingHole_Pad
- removed J15: Bus_M.2_Socket_M, A_HDJ_Library:PCIe_M.2_Connectors_P=0.5mm_H=4.2mm_KeyM, symbol Connector:Bus_M.2_Socket_M
- removed R27, R29: 0R/1%, A_HDJ_Library:R_0402_1005Metric, symbol Device:R
- removed R28: 0R/1%, Resistor_SMD:R_0402_1005Metric, symbol Device:R
- removed R30: 2.2K/1%, A_HDJ_Library:R_0402_1005Metric, symbol Device:R
- removed TP2: TestPoint, A_HDJ_Library:TestPoint_Pad_D1.5mm, symbol Connector:TestPoint
Connections:
- no-connect marks 50 -> 38
Other:
- note removed: "32.768kHz clock for low power mode"
- note removed: "SSD active LED"
- note removed: "To be grounded for SATA, No Connect for PCIe"
- company: DFRobot -> (none)
- title: Primer Carrier for LattePanda Mu -> Carrier for LattePanda Mu
