File: carrier_board.kicad_sch (KiCad schematic)
At the start: 6 parts

Commit message: Update KiCad carrier board project
Other:
- removed sheet GPIO
- removed sheet Gigabit Ethernet
- removed sheet PCIe x4
- sheet LattePanda Module ports: added none; removed HSIO_10_RX+, HSIO_10_RX-, HSIO_10_TX+, HSIO_10_TX-, HSIO_11_RX+, HSIO_11_RX-, HSIO_11_TX+, HSIO_11_TX-, HSIO_6_RX+, HSIO_6_RX-, HSIO_6_TX+, HSIO_6_TX-, HSIO_8_RX+, HSIO_8_RX-, HSIO_8_TX+, HSIO_8_TX-, HSIO_9_RX+, HSIO_9_RX-, HSIO_9_TX+, HSIO_9_TX-, I2C2_SCL, I2C2_SDA, I2C3_SCL, I2C3_SDA, I2C4_SCL, I2C4_SDA, I2C5_SCL, I2C5_SDA, REFCLK2+, REFCLK2-, REFCLK4+, REFCLK4-, SOC_UART0_RX, SOC_UART0_TX, SOC_UART1_RX, SOC_UART1_TX, SOC_UART2_RX, SOC_UART2_TX, ~{PEWAKE}, ~{PLT_RST}
- company: DFRobot -> (none)
- title: Primer Carrier for LattePanda Mu -> Carrier for LattePanda Mu
